Commit message: Updated  to use ros2_control first

File: src/my_bot/description/robot.urdf.xacro (robot description, xacro)
@@ -1,8 +1,15 @@
 <?xml version="1.0"?>
 <robot xmlns:xacro="http://www.ros.org/wiki/xacro"  name="robot">
+    <xacro:arg name="use_ros2_control" default="true"/>
     <xacro:include filename="inertial_macros.xacro" />
     <xacro:include filename="robot_core.xacro" />
+    <xacro:if value="$(arg use_ros2_control)">
+        <xacro:include filename="ros2_control.xacro"/>
+    </xacro:if>
+    <xacro:unless value="$(arg use_ros2_control)">
+        <xacro:include filename="gazebo_control.xacro"/>
+    </xacro:unless>
     <!-- <xacro:include filename="gazebo_control.xacro" /> -->
-    <xacro:include filename="ros2_control.xacro" />
+    <!-- <xacro:include filename="ros2_control.xacro" /> -->
     <xacro:include filename="lidar.xacro" />
 </robot>

File: src/my_bot/description/ros2_control.xacro (robot description, xacro)
@@ -5,5 +5,5 @@
             <plugin>gazebo_ros2_control/GazeboSystem</plugin>
         </hardware>
-        <joint name="left_wheel">
+        <joint name="left_wheel_joint">
             <command_interface name="velocity">
                 <param name="min">-10</param>
@@ -13,5 +13,5 @@
             <state_interface name="position"/>
         </joint>
-        <joint name="right_wheel">
+        <joint name="right_wheel_joint">
             <command_interface name="velocity">
                 <param name="min">-10</param>
